Commit message: Boom

File: cdrm_welding_support/urdf/irb2400_on_gantry.xacro.urdf (robot description, URDF)
Before this commit: robot irb_2400_on_gantry, 1 links, 1 joints
Links:
- added link boom_link
- added link carriage_link
Joints:
- removed joint base_robot_link
- added joint boom_joint: type prismatic, parent carriage_link, child boom_link, axis 0 0 -1, limit lower=0 upper=2 effort=0 velocity=0.5
- added joint boom_robot_joint: type fixed, parent boom_link, child robot_base_link, origin rpy=${pi} 0 0
- added joint track_joint: type prismatic, parent base_link, child carriage_link, axis 1 0 0, limit lower=0 upper=10 effort=0 velocity=1
