Commit message: Update example

File: cdrm_welding_support/urdf/m10ia_on_gantry.xacro.urdf (robot description, URDF)
Before this commit: robot m10ia_on_gantry, 6 links, 6 joints
Links:
- removed link boom_link_1
- removed link boom_link_2
- removed link carriage_link
- added link carriage_link_1; visual box size=0.25 4.25 0.25
- added link carriage_link_2
- added link carriage_link_3; visual box size=0.25 0.25 2
- link base_link: geometry visual box size=10 0.25 0.25; visual box size=10 0.25 0.25
Joints:
- removed joint boom_joint_1
- removed joint boom_joint_2
- removed joint boom_robot_joint
- removed joint track_joint
- added joint carriage_joint_1: type prismatic, parent base_link, child carriage_link_1, origin xyz=-5 0 0, axis 1 0 0, limit lower=0 upper=10 effort=0 velocity=1
- added joint carriage_joint_2: type prismatic, parent carriage_link_1, child carriage_link_2, axis 0 1 0, limit lower=-1.75 upper=1.75 effort=0 velocity=0.5
- added joint carriage_joint_3: type prismatic, parent carriage_link_2, child carriage_link_3, origin xyz=0.25 0 2.5, axis 0 0 1, limit lower=-1.5 upper=0 effort=0 velocity=0.5
- added joint carriange_robot_joint: type fixed, parent carriage_link_3, child robot_base_link, origin rpy=${pi} 0 0

Commit message: Nozzle

File: cdrm_welding_support/urdf/m10ia_on_gantry.xacro.urdf (robot description, URDF)
Before this commit: robot m10ia_on_gantry, 6 links, 6 joints
Links:
- added link nozzle_link; visual mesh filename=package://cdrm_welding_support/meshes/visual/nozzle_link.stl
Joints:
- added joint torch_nozzle_link: type fixed, parent torch_link, child nozzle_link
- joint torch_tcp_joint: origin xyz=0.02775225 0 0.21053771 rpy=0 ${radians(55)} 0 -> xyz=0.05636777 0 0.23057450 rpy=0 ${radians(55)} 0

Commit message: Continue welding CDRM generation

File: cdrm_welding_support/urdf/m10ia_on_gantry.xacro.urdf (robot description, URDF)
Before this commit: robot m10ia_on_gantry, 7 links, 7 joints
Links:
- link nozzle_link: geometry collision mesh filename=package://cdrm_welding_support/meshes/visual/nozzle_link.stl; visual mesh filename=package://cdrm_welding_support/meshes/visual/nozzle_link.stl
- link torch_link: geometry collision mesh filename=package://cdrm_welding_support/meshes/visual/torch_link.stl; visual mesh filename=package://cdrm_welding_support/meshes/visual/torch_link.stl
Joints:
- removed joint carriange_robot_joint
- added joint carriage_robot_joint: type fixed, parent carriage_link_3, child robot_base_link, origin rpy=${pi} 0 0

Commit message: Add L profile

File: cdrm_welding_support/urdf/m10ia_on_gantry.xacro.urdf (robot description, URDF)
Before this commit: robot m10ia_on_gantry, 7 links, 7 joints
Links:
- added link workpiece_link; collision mesh filename=package://cdrm_welding_support/meshes/l_profile.stl; visual mesh filename=package://cdrm_welding_support/meshes/l_profile.stl
Joints:
- added joint base_workpiece_joint: type fixed, parent base_link, child workpiece_link
