Commit message: Rename package

File: cdrm_welding_tutorial/urdf/m10ia_on_gantry.xacro.urdf (robot description, URDF)
Before this commit: robot m10ia_on_gantry, 8 links, 8 joints
Links:
- link nozzle_link: geometry collision mesh filename=package://cdrm_welding_tutorial/meshes/visual/nozzle_link.s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; visual mesh filename=package://cdrm_welding_tutorial/meshes/visual/nozzle_link.s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
- link torch_link: geometry collision mesh filename=package://cdrm_welding_tutorial/meshes/visual/torch_link.stl; visual mesh filename=package://cdrm_welding_tutorial/meshes/visual/torch_link.stl
- link workpiece_link: geometry collision mesh filename=package://cdrm_welding_tutorial/meshes/l_profile.stl; visual mesh filename=package://cdrm_welding_tutorial/meshes/l_profile.stl

Commit message: Invoke robot CDRM generator

File: cdrm_welding_tutorial/urdf/m10ia_on_gantry.xacro.urdf (robot description, URDF)
Before this commit: robot m10ia_on_gantry, 8 links, 8 joints
Links:
- removed link tcp_link
- link workpiece_link: geometry 
Joints:
- removed joint torch_tcp_joint
- joint torch_nozzle_link: origin (none) -> xyz=0.05636777 0 0.23057450 rpy=0 ${radians(55)} 0

Commit message: Make single rail

File: cdrm_welding_tutorial/urdf/m10ia_on_gantry.xacro.urdf (robot description, URDF)
Before this commit: robot m10ia_on_gantry, 7 links, 7 joints
Links:
- link base_link: geometry visual box size=10 0.25 0.25
Joints:
- joint carriage_joint_1: limit lower=0 upper=10 effort=0 velocity=1 -> lower=0 upper=5 effort=0 velocity=1
- joint carriage_joint_2: limit lower=-1.75 upper=1.75 effort=0 velocity=0.5 -> lower=-1 upper=1 effort=0 velocity=0.5

Commit message: Update robot model

File: cdrm_welding_tutorial/urdf/m10ia_on_gantry.xacro.urdf (robot description, URDF)
Before this commit: robot m10ia_on_gantry, 7 links, 7 joints
Links:
- link base_link: geometry visual box size=10 0.1 0.4; visual box size=10 0.1 0.4
- link carriage_link_1: geometry visual box size=0.4 3.5 0.4; visual box size=0.8 0.8 3.25
Joints:
- joint carriage_joint_3: limit lower=-1.5 upper=0 effort=0 velocity=0.5 -> lower=-1.3 upper=0 effort=0 velocity=0.5; origin xyz=0.25 0 2.5 -> xyz=0.35 0 2.5

Commit message: Put workpiece in the URDF

File: cdrm_welding_tutorial/urdf/m10ia_on_gantry.xacro.urdf (robot description, URDF)
Before this commit: robot m10ia_on_gantry, 7 links, 7 joints
Links:
- link workpiece_link: geometry collision mesh filename=package://cdrm_welding_tutorial/meshes/l_profile.stl; visual mesh filename=package://cdrm_welding_tutorial/meshes/l_profile.stl
