Commit message: Use full states and remove interial

File: example_quadruped_description/urdf/body.urdf.xacro (robot description, xacro)
@@ -10,9 +10,4 @@
         <geometry><mesh filename="package://example_quadruped_description/meshes/body_link.stl" /></geometry>
       </collision>
-      <inertial>
-        <origin xyz="-7.0772E-05 0.022175 0.00069238" />
-        <mass value="0.86768" />
-        <inertia ixx="0.004313" ixy="7.3571E-06" ixz="-4.1802E-06" iyy="0.0063166" iyz="1.4712E-05" izz="0.0027301" />
-      </inertial>
     </link>
     <joint name="body_joint" type="fixed">

File: example_quadruped_description/urdf/leg.urdf.xacro (robot description, xacro)
@@ -24,9 +24,4 @@
         <origin rpy="${-pi / 2} 0 ${pi / 2}" />
       </collision>
-      <inertial>
-        <origin xyz="0.0028255 0.016487 -0.038239" />
-        <mass value="0.054025" />
-        <inertia ixx="4.2638E-05" ixy="-1.8883E-07" ixz="-4.2377E-06" iyy="5.3271E-05" iyz="2.555E-06" izz="2.8624E-05" />
-      </inertial>
     </link>
     <link name="${name}_femur_link">
@@ -40,9 +35,4 @@
         <origin rpy="0 0 ${-pi / 2}" />
       </collision>
-      <inertial>
-        <origin xyz="4.1633E-17 0.0545 -0.0002317" />
-        <mass value="0.18426" />
-        <inertia ixx="0.00033345" ixy="-6.5254E-08" ixz="-1.5302E-19" iyy="4.8055E-05" iyz="-2.3378E-19" izz="0.0003165" />
-      </inertial>
     </link>
     <link name="${name}_tibia_link">
@@ -56,9 +46,4 @@
         <origin rpy="${-pi / 2} ${-pi / 2} 0" />
       </collision>
-      <inertial>
-        <origin xyz="-0.001867 0.094612 7.7874E-06" />
-        <mass value="0.08176" />
-        <inertia ixx="0.0009073" ixy="1.4442E-05" ixz="1.1866E-09" iyy="2.5535E-05" iyz="9.4278E-08" izz="0.00092384" />
-      </inertial>
     </link>
     <link name="${name}_foot_link" />
