Commit message: Reduce range

File: example_quadruped_description/urdf/leg.urdf.xacro (robot description, xacro)
@@ -53,5 +53,5 @@
       <xacro:insert_block name="origin" />
       <axis xyz="0 0 1" />
-      <limit lower="-1.8326" upper="1.8326" effort="3.1" velocity="7" />
+      <limit lower="-1.0472" upper="1.0472" effort="3.1" velocity="7" />
     </joint>
     <joint name="${name}_femur_joint" type="revolute">

Commit message: Adjust joint limits

File: example_quadruped_description/urdf/leg.urdf.xacro (robot description, xacro)
@@ -53,5 +53,5 @@
       <xacro:insert_block name="origin" />
       <axis xyz="0 0 1" />
-      <limit lower="-1.0472" upper="1.0472" effort="3.1" velocity="7" />
+      <limit lower="-0.785398" upper="0.785398" effort="3.1" velocity="7" />
     </joint>
     <joint name="${name}_femur_joint" type="revolute">
